File: oni-base/oni-base.kicad_pcb (KiCad board)
At the start: 2 copper layers, 113.3 x 89.7 mm, 3 parts

Commit message: added text and images
Parts:
- added  : LOGO, LOGO, F.Cu at (73.0, 103.0)
- added  : LOGO, LOGO, B.Cu at (78.5, 103.0)
Other:
- board text added: "#!/usr/bin/env"
- board text added: "ラム"
- board text added: "レム"
