File: oni-kb/oni-kb.kicad_pcb (KiCad board)
At the start: 2 copper layers, 113.3 x 89.7 mm, 37 parts, among them J1 JST-BATTERY, SW1 SW_Push, SW10 SW_Push, SW11 SW_Push, SW12 SW_Push, SW14 SW_Push, SW15 SW_Push, SW16 SW_Push, SW17 SW_Push, SW18 SW_Push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

Commit message: added text and images
Parts:
- moved   1.12 mm to (127.0, 117.6)

Commit message: readme images
Parts:
- removed the REF** at (93.3, 70.3) (x2)
Other:
- board text added: "____"
- board text added: "Øni"
- board text added: "鬼"
